Commit message: Configure ZED stereo image output for FlowNav

File: cat_bringup/urdf/experiment_robot.urdf.xacro (robot description, xacro)
@@ -68,10 +68,10 @@
   </joint>
   <!-- RPLIDAR S1 scan origin (rotating laser axis), not its bottom mounting face.
-       Measured from base_link: 8 mm forward, centered, 192 mm above ground. -->
+       Measured from base_link: 33.19 mm forward, centered, 248.83 mm above ground. -->
   <link name="laser"/>
   <joint name="laser_joint" type="fixed">
     <parent link="base_link"/><child link="laser"/>
     <!-- The scanner's +X direction faces the rear of the vehicle. -->
-    <origin xyz="0.008 0 0.192" rpy="0 0 ${pi}"/>
+    <origin xyz="0.03319 0 0.24883" rpy="0 0 ${pi}"/>
   </joint>
   <!-- Camera mounting reference is now on the robot centerline (y=0).

Commit message: Update ZED camera mount pose

File: cat_bringup/urdf/experiment_robot.urdf.xacro (robot description, xacro)
@@ -75,6 +75,6 @@
     <origin xyz="0.03319 0 0.24883" rpy="0 0 ${pi}"/>
   </joint>
-  <!-- Camera mounting reference is now on the robot centerline (y=0).
-       Previous longitudinal position and mounting height are retained. -->
+  <!-- Camera mount: 285 mm behind the axle, centered, 550 mm above ground.
+       Positive pitch tips the forward-facing camera down by 12 degrees. -->
   <xacro:include filename="$(find zed_description)/urdf/zed_macro.urdf.xacro"/>
   <xacro:zed_camera name="zed" model="zedm" enable_gnss="false">
@@ -83,5 +83,5 @@
   <joint name="zed_mount_joint" type="fixed">
     <parent link="base_link"/><child link="zed_camera_link"/>
-    <origin xyz="-0.270 0 0.54675" rpy="0 0 0"/>
+    <origin xyz="-0.285 0 0.550" rpy="0 ${12*pi/180} 0"/>
   </joint>
   <!-- GNSS link origin is the user-provided antenna reference point. -->

Commit message: Support LiDAR-only navigation without ZED packages

File: cat_bringup/urdf/experiment_robot.urdf.xacro (robot description, xacro)
@@ -1,4 +1,5 @@
 <?xml version="1.0"?>
 <robot name="experiment_robot" xmlns:xacro="http://www.ros.org/wiki/xacro">
+  <xacro:arg name="use_zed" default="true"/>
   <!-- Measurements are expressed from the drive-axle midpoint at ground level. -->
   <xacro:property name="wheel_radius" value="0.050"/>
@@ -77,12 +78,14 @@
   <!-- Camera mount: 285 mm behind the axle, centered, 550 mm above ground.
        Positive pitch tips the forward-facing camera down by 12 degrees. -->
-  <xacro:include filename="$(find zed_description)/urdf/zed_macro.urdf.xacro"/>
-  <xacro:zed_camera name="zed" model="zedm" enable_gnss="false">
-    <origin xyz="0 0 0" rpy="0 0 0"/>
-  </xacro:zed_camera>
-  <joint name="zed_mount_joint" type="fixed">
-    <parent link="base_link"/><child link="zed_camera_link"/>
-    <origin xyz="-0.285 0 0.550" rpy="0 ${12*pi/180} 0"/>
-  </joint>
+  <xacro:if value="$(arg use_zed)">
+    <xacro:include filename="$(find zed_description)/urdf/zed_macro.urdf.xacro"/>
+    <xacro:zed_camera name="zed" model="zedm" enable_gnss="false">
+      <origin xyz="0 0 0" rpy="0 0 0"/>
+    </xacro:zed_camera>
+    <joint name="zed_mount_joint" type="fixed">
+      <parent link="base_link"/><child link="zed_camera_link"/>
+      <origin xyz="-0.285 0 0.550" rpy="0 ${12*pi/180} 0"/>
+    </joint>
+  </xacro:if>
   <!-- GNSS link origin is the user-provided antenna reference point. -->
   <link name="gnss_antenna_link">

Commit message: Add VLP-16 sensor bringup and LiDAR selection

File: cat_bringup/urdf/experiment_robot.urdf.xacro (robot description, xacro)
@@ -2,4 +2,8 @@
 <robot name="experiment_robot" xmlns:xacro="http://www.ros.org/wiki/xacro">
   <xacro:arg name="use_zed" default="true"/>
+  <xacro:arg name="rplidar_x" default="0.03319"/>
+  <xacro:arg name="rplidar_y" default="0"/>
+  <xacro:arg name="rplidar_z" default="0.24883"/>
+  <xacro:arg name="rplidar_yaw" default="3.141592653589793"/>
   <!-- Measurements are expressed from the drive-axle midpoint at ground level. -->
   <xacro:property name="wheel_radius" value="0.050"/>
@@ -68,11 +72,16 @@
     <parent link="base_link"/><child link="safety_footprint_link"/>
   </joint>
-  <!-- RPLIDAR S1 scan origin (rotating laser axis), not its bottom mounting face.
-       Measured from base_link: 33.19 mm forward, centered, 248.83 mm above ground. -->
+  <!-- RPLIDAR S1 scan origin. Defaults preserve the previous measured mount. -->
   <link name="laser"/>
   <joint name="laser_joint" type="fixed">
     <parent link="base_link"/><child link="laser"/>
-    <!-- The scanner's +X direction faces the rear of the vehicle. -->
-    <origin xyz="0.03319 0 0.24883" rpy="0 0 ${pi}"/>
+    <origin xyz="$(arg rplidar_x) $(arg rplidar_y) $(arg rplidar_z)"
+            rpy="0 0 $(arg rplidar_yaw)"/>
+  </joint>
+  <!-- VLP-16 laser reference, 18.6 mm forward and 207 mm high, tilted down 7 deg. -->
+  <link name="vlp16"/>
+  <joint name="vlp16_joint" type="fixed">
+    <parent link="base_link"/><child link="vlp16"/>
+    <origin xyz="0.0186 0 0.207" rpy="0 ${7*pi/180} 0"/>
   </joint>
   <!-- Camera mount: 285 mm behind the axle, centered, 550 mm above ground.

Commit message: Define front and rear RPLIDAR mounts

File: cat_bringup/urdf/experiment_robot.urdf.xacro (robot description, xacro)
@@ -6,4 +6,5 @@
   <xacro:arg name="rplidar_z" default="0.24883"/>
   <xacro:arg name="rplidar_yaw" default="3.141592653589793"/>
+  <xacro:arg name="rplidar_roll" default="0"/>
   <!-- Measurements are expressed from the drive-axle midpoint at ground level. -->
   <xacro:property name="wheel_radius" value="0.050"/>
@@ -72,10 +73,20 @@
     <parent link="base_link"/><child link="safety_footprint_link"/>
   </joint>
-  <!-- RPLIDAR S1 scan origin. Defaults preserve the previous measured mount. -->
-  <link name="laser"/>
-  <joint name="laser_joint" type="fixed">
-    <parent link="base_link"/><child link="laser"/>
+  <!-- RPLIDAR S1 mounting positions; /scan uses the selected frame only. -->
+  <link name="RPLIDAR_F"/>
+  <joint name="RPLIDAR_F_joint" type="fixed">
+    <parent link="base_link"/><child link="RPLIDAR_F"/>
+    <origin xyz="0.03319 0 0.24883" rpy="0 0 ${pi}"/>
+  </joint>
+  <link name="RPLIDAR_B"/>
+  <joint name="RPLIDAR_B_joint" type="fixed">
+    <parent link="base_link"/><child link="RPLIDAR_B"/>
+    <origin xyz="-0.3095 0 0.49735" rpy="${pi} 0 ${-pi/2}"/>
+  </joint>
+  <link name="RPLIDAR_custom"/>
+  <joint name="RPLIDAR_custom_joint" type="fixed">
+    <parent link="base_link"/><child link="RPLIDAR_custom"/>
     <origin xyz="$(arg rplidar_x) $(arg rplidar_y) $(arg rplidar_z)"
-            rpy="0 0 $(arg rplidar_yaw)"/>
+            rpy="$(arg rplidar_roll) 0 $(arg rplidar_yaw)"/>
   </joint>
   <!-- VLP-16 laser reference, 18.6 mm forward and 207 mm high, tilted down 7 deg. -->

Commit message: Correct rear RPLIDAR heading

File: cat_bringup/urdf/experiment_robot.urdf.xacro (robot description, xacro)
@@ -82,5 +82,5 @@
   <joint name="RPLIDAR_B_joint" type="fixed">
     <parent link="base_link"/><child link="RPLIDAR_B"/>
-    <origin xyz="-0.3095 0 0.49735" rpy="${pi} 0 ${-pi/2}"/>
+    <origin xyz="-0.3095 0 0.49735" rpy="${pi} 0 ${pi/2}"/>
   </joint>
   <link name="RPLIDAR_custom"/>

Commit message: Add front and rear VLP-16 mounts

File: cat_bringup/urdf/experiment_robot.urdf.xacro (robot description, xacro)
@@ -90,9 +90,14 @@
             rpy="$(arg rplidar_roll) 0 $(arg rplidar_yaw)"/>
   </joint>
-  <!-- VLP-16 laser reference, 18.6 mm forward and 207 mm high, tilted down 7 deg. -->
-  <link name="vlp16"/>
-  <joint name="vlp16_joint" type="fixed">
-    <parent link="base_link"/><child link="vlp16"/>
+  <!-- VLP-16 front and rear mounting positions. -->
+  <link name="VLP16_F"/>
+  <joint name="VLP16_F_joint" type="fixed">
+    <parent link="base_link"/><child link="VLP16_F"/>
     <origin xyz="0.0186 0 0.207" rpy="0 ${7*pi/180} 0"/>
+  </joint>
+  <link name="VLP16_B"/>
+  <joint name="VLP16_B_joint" type="fixed">
+    <parent link="base_link"/><child link="VLP16_B"/>
+    <origin xyz="-0.347981 0 0.515158" rpy="${pi} ${20*pi/180} ${pi/2}"/>
   </joint>
   <!-- Camera mount: 285 mm behind the axle, centered, 550 mm above ground.

Commit message: Align VLP-16 pitch toward robot front

File: cat_bringup/urdf/experiment_robot.urdf.xacro (robot description, xacro)
@@ -99,5 +99,5 @@
   <joint name="VLP16_B_joint" type="fixed">
     <parent link="base_link"/><child link="VLP16_B"/>
-    <origin xyz="-0.347981 0 0.515158" rpy="${pi} ${20*pi/180} ${pi/2}"/>
+    <origin xyz="-0.347981 0 0.515158" rpy="${(180-20)*pi/180} 0 ${pi/2}"/>
   </joint>
   <!-- Camera mount: 285 mm behind the axle, centered, 550 mm above ground.

Commit message: Reverse VLP-16 forward pitch direction

File: cat_bringup/urdf/experiment_robot.urdf.xacro (robot description, xacro)
@@ -99,5 +99,5 @@
   <joint name="VLP16_B_joint" type="fixed">
     <parent link="base_link"/><child link="VLP16_B"/>
-    <origin xyz="-0.347981 0 0.515158" rpy="${(180-20)*pi/180} 0 ${pi/2}"/>
+    <origin xyz="-0.347981 0 0.515158" rpy="${(180+20)*pi/180} 0 ${pi/2}"/>
   </joint>
   <!-- Camera mount: 285 mm behind the axle, centered, 550 mm above ground.

Commit message: Reverse VLP-16 yaw direction

File: cat_bringup/urdf/experiment_robot.urdf.xacro (robot description, xacro)
@@ -99,5 +99,5 @@
   <joint name="VLP16_B_joint" type="fixed">
     <parent link="base_link"/><child link="VLP16_B"/>
-    <origin xyz="-0.347981 0 0.515158" rpy="${(180+20)*pi/180} 0 ${pi/2}"/>
+    <origin xyz="-0.347981 0 0.515158" rpy="${(180-20)*pi/180} 0 ${-pi/2}"/>
   </joint>
   <!-- Camera mount: 285 mm behind the axle, centered, 550 mm above ground.

Commit message: Update RPLIDAR front mount position

File: cat_bringup/urdf/experiment_robot.urdf.xacro (robot description, xacro)
@@ -2,7 +2,7 @@
 <robot name="experiment_robot" xmlns:xacro="http://www.ros.org/wiki/xacro">
   <xacro:arg name="use_zed" default="true"/>
-  <xacro:arg name="rplidar_x" default="0.03319"/>
+  <xacro:arg name="rplidar_x" default="0.00319"/>
   <xacro:arg name="rplidar_y" default="0"/>
-  <xacro:arg name="rplidar_z" default="0.24883"/>
+  <xacro:arg name="rplidar_z" default="0.25435"/>
   <xacro:arg name="rplidar_yaw" default="3.141592653589793"/>
   <xacro:arg name="rplidar_roll" default="0"/>
@@ -77,5 +77,5 @@
   <joint name="RPLIDAR_F_joint" type="fixed">
     <parent link="base_link"/><child link="RPLIDAR_F"/>
-    <origin xyz="0.03319 0 0.24883" rpy="0 0 ${pi}"/>
+    <origin xyz="0.00319 0 0.25435" rpy="0 0 ${pi}"/>
   </joint>
   <link name="RPLIDAR_B"/>

Commit message: Move front RPLiDAR mount forward by 30 mm

File: cat_bringup/urdf/experiment_robot.urdf.xacro (robot description, xacro)
@@ -2,5 +2,5 @@
 <robot name="experiment_robot" xmlns:xacro="http://www.ros.org/wiki/xacro">
   <xacro:arg name="use_zed" default="true"/>
-  <xacro:arg name="rplidar_x" default="0.00319"/>
+  <xacro:arg name="rplidar_x" default="0.03319"/>
   <xacro:arg name="rplidar_y" default="0"/>
   <xacro:arg name="rplidar_z" default="0.25435"/>
@@ -77,5 +77,5 @@
   <joint name="RPLIDAR_F_joint" type="fixed">
     <parent link="base_link"/><child link="RPLIDAR_F"/>
-    <origin xyz="0.00319 0 0.25435" rpy="0 0 ${pi}"/>
+    <origin xyz="0.03319 0 0.25435" rpy="0 0 ${pi}"/>
   </joint>
   <link name="RPLIDAR_B"/>
